File: FSK Project.kicad_pcb (KiCad board)
At the start: 2 copper layers, 85.5 x 62 mm, 60 parts, among them J1 DATA IN, J2 TX_PAIR, J3 RX_PAIR, J4 DATA_OUT, Q1 2N3904, Q2 2N3904, SW1 MAN, U1 MC14046BCP, U2 LM393, U3 MC14046BCP

Commit message: Add final libs, include last leftover bits, fix op-amp and verify on board
Parts:
- added D2: RX, LED_THT:LED_D3.0mm, F.Cu at (158.7, 85.4)
- added G***: LOGO, KenwoodFox:KITSUNE_LOGO, F.Cu at (145.0, 116.5)
- added G***: LOGO, thermocline:monk, B.Cu at (158.5, 96.5)
- added R22: 100K, Resistor_THT:R_Axial_DIN0204_L3.6mm_D1.6mm_P7.62mm_Horizontal, F.Cu at (181.5, 127.8)
- added R23: 150R, Resistor_THT:R_Axial_DIN0204_L3.6mm_D1.6mm_P7.62mm_Horizontal, F.Cu at (156.2, 82.0)
- added REF**: OSHW-Logo2_9.8x8mm_Copper, Symbol:OSHW-Logo2_9.8x8mm_Copper, F.Cu at (159.0, 94.5)
- added REF**: OSHW-Logo2_9.8x8mm_Copper, Symbol:OSHW-Logo2_9.8x8mm_Copper, F.Cu at (136.5, 97.5)
- added SNHU_NEW***: LOGO, KenwoodFox:SNHU_NEW, B.Cu at (141.0, 128.5)
- added SNHU_NEW***: LOGO, KenwoodFox:SNHU_NEW, B.Cu at (163.0, 74.0)
- R17: value 100K -> 300K
Connections:
- RV1 pad 2: Net-(U2A-+) -> Net-(U2A--)
- U2 pad 2: /DEM_OUT -> Net-(U2A--)
Routing:
- net /DATA_OUT: track 42.7 -> 59.0 mm
- net Net-(U2A--): track 0.00 -> 11.6 mm
- net Net-(D2-A): track 0.00 -> 3.41 mm
- net Net-(U2A-+): track 25.1 -> 28.1 mm
- net /DEM_OUT: track 51.5 -> 54.4 mm
- net GND: track 6.39 -> 8.10 mm
Other:
- board text added: "RECEIVE"
- board text added: "TRANSMIT"
- board text added: "Use TTL 5V Be kind to yourself"
