File: FSK Project.kicad_pcb (KiCad board)
At the start: 2 copper layers, 85.5 x 62 mm, 69 parts, among them J1 DATA IN, J2 TX_PAIR, J3 RX_PAIR, J4 DATA_OUT, Q1 2N3904, Q2 2N3904, SW1 MAN, U1 MC14046BCP, U2 LM393, U3 MC14046BCP

Commit message: fix some issues i made in the design oops
Parts:
- R13, R3: value 33K -> 100k
Connections:
- R21 pad 1: Net-(U3-SigIn) -> /MOD_IN
- TP3 pad 1: Net-(U3-SigIn) -> /MOD_IN
- U3 pad 14: Net-(U3-SigIn) -> Net-(U3-FOUT)
- U3 pad 3: Net-(U3-FOUT) -> /MOD_IN
Routing:
- net /MOD_IN: track 0.00 -> 43.2 mm, vias 0 -> 2
- net Net-(U3-SigIn): track 40.5 -> 0.00 mm
- net Net-(U3-FOUT): track 11.3 -> 9.05 mm
Changed lines of the file:
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@@
 			)
 		)
-		(attr exclude_from_bom)
+		(attr exclude_from_bom dnp)
 		(duplicate_pad_numbers_are_jumpers no)
 		(fp_circle
@@
 			)
 		)
-		(attr exclude_from_bom)
+		(attr exclude_from_bom dnp)
 		(duplicate_pad_numbers_are_jumpers no)
 		(fp_circle
@@
 			(layers "*.Cu" "*.Mask")
 			(remove_unused_layers no)
-			(net "Net-(U3-SigIn)")
+			(net "/MOD_IN")
 			(pinfunction "1_1")
 			(pintype "passive")
@@
 			)
 		)
-		(property "Value" "33K"
+		(property "Value" "100k"
 			(at 3.81 1.92 0)
 			(layer "F.Fab")
@@
 			(layers "*.Cu" "*.Mask")
 			(remove_unused_layers no)
-			(net "Net-(U3-SigIn)")
+			(net "/MOD_IN")
 			(pintype "passive")
 		)
@@
 			)
 		)
-		(property "Value" "33K"
+		(property "Value" "100k"
 			(at 3.81 1.92 90)
 			(layer "F.Fab")
@@
 			(layers "*.Cu" "*.Mask")
 			(remove_unused_layers no)
-			(net "Net-(U3-FOUT)")
+			(net "/MOD_IN")
 			(pinfunction "RefIn_3")
 			(pintype "input")
@@
 			(layers "*.Cu" "*.Mask")
 			(remove_unused_layers no)
-			(net "Net-(U3-SigIn)")
+			(net "Net-(U3-FOUT)")
 			(pinfunction "SigIn_14")
 			(pintype "input")
@@
 			)
 		)
-		(attr exclude_from_bom)
+		(attr exclude_from_bom dnp)
 		(duplicate_pad_numbers_are_jumpers no)
 		(fp_circle
@@
 			)
 		)
-		(attr exclude_from_bom)
+		(attr exclude_from_bom dnp)
 		(duplicate_pad_numbers_are_jumpers no)
 		(fp_circle
@@
 	)
 	(segment
-		(start 167.5 85.5)
-		(end 172 85.5)
-		(width 1.4)
-		(layer "B.Cu")
-		(net "Net-(U3-SigIn)")
-	)
-	(segment
-		(start 177.31 93.69)
-		(end 177.69 93.69)
-		(width 1.4)
-		(layer "B.Cu")
-		(net "Net-(U3-SigIn)")
-	)
-	(segment
-		(start 174 87.5)
-		(end 174 91.572082)
-		(width 1.4)
-		(layer "B.Cu")
-		(net "Net-(U3-SigIn)")
-	)
-	(segment
-		(start 177.69 93.69)
-		(end 181 97)
-		(width 1.4)
-		(layer "B.Cu")
-		(net "Net-(U3-SigIn)")
-	)
-	(segment
-		(start 191.5 99.5)
-		(end 191.5 102.5)
-		(width 1.4)
-		(layer "B.Cu")
-		(net "Net-(U3-SigIn)")
-	)
-	(segment
-		(start 181 97)
-		(end 189 97)
-		(width 1.4)
-		(layer "B.Cu")
-		(net "Net-(U3-SigIn)")
-	)
-	(segment
-		(start 165.5 87.5)
-		(end 167.5 85.5)
-		(width 1.4)
-		(layer "B.Cu")
-		(net "Net-(U3-SigIn)")
-	)
-	(segment
-		(start 172 85.5)
-		(end 174 87.5)
-		(width 1.4)
-		(layer "B.Cu")
-		(net "Net-(U3-SigIn)")
-	)
-	(segment
-		(start 176.117918 93.69)
-		(end 177.31 93.69)
-		(width 1.4)
-		(layer "B.Cu")
-		(net "Net-(U3-SigIn)")
-	)
-	(segment
-		(start 189 97)
-		(end 191.5 99.5)
-		(width 1.4)
-		(layer "B.Cu")
-		(net "Net-(U3-SigIn)")
-	)
-	(segment
-		(start 174 91.572082)
-		(end 176.117918 93.69)
-		(width 1.4)
-		(layer "B.Cu")
-		(net "Net-(U3-SigIn)")
-	)
-	(segment
-		(start 165.5 90)
-		(end 165.5 87.5)
-		(width 1.4)
-		(layer "B.Cu")
-		(net "Net-(U3-SigIn)")
-	)
-	(segment
 		(start 124 98.5)
 		(end 124 108)
@@
 	)
 	(segment
-		(start 165 94.19)
-		(end 165.5 93.69)
+		(start 177.31 93.69)
+		(end 177.69 93.69)
 		(width 1.4)
-		(layer "F.Cu")
+		(layer "B.Cu")
 		(net "Net-(U3-FOUT)")
 	)
 	(segment
-		(start 165.5 96.23)
-		(end 165 95.73)
+		(start 175.31 93.69)
+		(end 177.31 93.69)
 		(width 1.4)
-		(layer "F.Cu")
+		(layer "B.Cu")
 		(net "Net-(U3-FOUT)")
 	)
 	(segment
-		(start 165 95.73)
-		(end 165 94.19)
+		(start 172.77 96.23)
+		(end 175.31 93.69)
 		(width 1.4)
-		(layer "F.Cu")
+		(layer "B.Cu")
 		(net "Net-(U3-FOUT)")
 	)
 	(segment
 		(start 169.69 96.23)
-		(end 165.5 96.23)
+		(end 172.77 96.23)
 		(width 1.4)
-		(layer "F.Cu")
+		(layer "B.Cu")
 		(net "Net-(U3-FOUT)")
 	)
 	(segment
-		(start 165.5 93.69)
-		(end 169.69 93.69)
+		(start 185.5 92)
+		(end 179.5 86)
 		(width 1.4)
 		(layer "F.Cu")
-		(net "Net-(U3-FOUT)")
+		(net "/MOD_IN")
+	)
+	(segment
+		(start 188 97)
+		(end 185.5 94.5)
+		(width 1.4)
+		(layer "F.Cu")
+		(net "/MOD_IN")
+	)
+	(segment
+		(start 185.5 94.5)
+		(end 185.5 92)
+		(width 1.4)
+		(layer "F.Cu")
+		(net "/MOD_IN")
+	)
+	(via
+		(at 188 97)
+		(size 0.6)
+		(drill 0.3)
+		(layers "F.Cu" "B.Cu")
+		(net "/MOD_IN")
+	)
+	(via
+		(at 179.5 86)
+		(size 0.6)
+		(drill 0.3)
+		(layers "F.Cu" "B.Cu")
+		(net "/MOD_IN")
+	)
+	(segment
+		(start 173.5 92.5)
+		(end 173.5 89)
+		(width 1.4)
+		(layer "B.Cu")
+		(net "/MOD_IN")
+	)
+	(segment
+		(start 168.19 93.69)
+		(end 169.69 93.69)
+		(width 1.4)
+		(layer "B.Cu")
+		(net "/MOD_IN")
+	)
+	(segment
+		(start 165.5 91)
+		(end 168.19 93.69)
+		(width 1.4)
+		(layer "B.Cu")
+		(net "/MOD_IN")
+	)
+	(segment
+		(start 173.5 89)
+		(end 176.5 86)
+		(width 1.4)
+		(layer "B.Cu")
+		(net "/MOD_IN")
+	)
+	(segment
+		(start 191.5 99.927258)
+		(end 188.572742 97)
+		(width 1.4)
+		(layer "B.Cu")
+		(net "/MOD_IN")
+	)
+	(segment
+		(start 188.572742 97)
+		(end 188 97)
+		(width 1.4)
+		(layer "B.Cu")
+		(net "/MOD_IN")
+	)
+	(segment
+		(start 165.5 90)
+		(end 165.5 91)
+		(width 1.4)
+		(layer "B.Cu")
+		(net "/MOD_IN")
+	)
+	(segment
+		(start 191.5 102.5)
+		(end 191.5 99.927258)
+		(width 1.4)
+		(layer "B.Cu")
+		(net "/MOD_IN")
+	)
+	(segment
+		(start 176.5 86)
+		(end 179.5 86)
+		(width 1.4)
+		(layer "B.Cu")
+		(net "/MOD_IN")
+	)
+	(segment
+		(start 169.69 93.69)
+		(end 172.31 93.69)
+		(width 1.4)
+		(layer "B.Cu")
+		(net "/MOD_IN")
+	)
+	(segment
+		(start 172.31 93.69)
+		(end 173.5 92.5)
+		(width 1.4)
+		(layer "B.Cu")
+		(net "/MOD_IN")
 	)
 	(zone
